File: hardware/sahel_pcb_main/mcu.kicad_sch (KiCad schematic)
At the start: 35 parts, among them J301 JTAG_SWD, J302 USB_C_Receptacle_USB2.0_16P, SW301 BOOT, SW302 RESET, U301 STM32H7B0VBTx, X301 8MHz

Commit message: docs: advance README documentation
Refactor code structure for improved readability and maintainability
Connections:
- net Bat_Alert: now reaches U301.1 (PE2)
- no-connect marks 34 -> 33
Changed lines of the file:
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@@
-	)
-	(no_connect
-		(at 55.88 71.12)
 	)
 	(no_connect
@@
 		)
 	)
+	(hierarchical_label "Bat_Alert"
+		(shape input)
+		(at 55.88 71.12 180)
+		(effects
+			(font
+				(size 1.27 1.27)
+			)
+			(justify right)
+		)
+	)
