File: hardware/sahel_pcb_main/sahel_pcb.kicad_sch (KiCad schematic)
At the start: 2 parts, among them J101 Conn_02x26_Odd_Even, J102 Conn_02x26_Odd_Even

Commit message: docs: advance README documentation
Refactor code structure for improved readability and maintainability
Parts:
- added J103: Batt, Connector_JST:JST_ZH_B4B-ZR_1x04_P1.50mm_Vertical, symbol Connector:Conn_01x04_Pin
Connections:
- net 3.3V_MAIN: now also J103.4 (Pin_4)
- new net _SCL: J103.3 (Pin_3)
- new net _SDA: J103.2 (Pin_2)
- new net bat_alert: J103.1 (Pin_1)
Other:
- sheet MCU ports: added Bat_Alert; removed none
Changed lines of the file:
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@@
+	(wire
+		(pts
+			(xy 173.99 27.94) (xy 199.39 27.94)
+		)
+		(stroke
+			(width 0)
+			(type default)
+		)
+	)
 	(wire
 		(pts
@@
 		)
 	)
+	(label "_SCL"
+		(at 173.99 25.4 0)
+		(effects
+			(font
+				(size 1.27 1.27)
+			)
+			(justify left bottom)
+		)
+	)
 	(label "DRDY_M"
 		(at 81.28 33.02 90)
@@
 		)
 	)
+	(label "_SDA"
+		(at 114.3 60.96 0)
+		(effects
+			(font
+				(size 1.27 1.27)
+			)
+			(justify left bottom)
+		)
+	)
 	(label "BUS_RS_A"
 		(at 152.4 29.21 90)
@@
 		)
 	)
+	(label "bat_alert"
+		(at 173.99 20.32 0)
+		(effects
+			(font
+				(size 1.27 1.27)
+			)
+			(justify left bottom)
+		)
+	)
 	(label "BUS_SCL"
 		(at 236.22 68.58 0)
@@
 		)
 	)
+	(label "_SDA"
+		(at 173.99 22.86 0)
+		(effects
+			(font
+				(size 1.27 1.27)
+			)
+			(justify left bottom)
+		)
+	)
+	(label "_SCL"
+		(at 114.3 58.42 0)
+		(effects
+			(font
+				(size 1.27 1.27)
+			)
+			(justify left bottom)
+		)
+	)
 	(label "BUS_SDA"
 		(at 236.22 45.72 0)
@@
 		)
 	)
+	(label "bat_alert"
+		(at 91.44 33.02 90)
+		(effects
+			(font
+				(size 1.27 1.27)
+			)
+			(justify left bottom)
+		)
+	)
 	(label "SPI_MOSI"
 		(at 223.52 45.72 180)
@@
 			)
 			(justify right bottom)
+		)
+	)
+	(symbol
+		(lib_id "Connector:Conn_01x04_Pin")
+		(at 168.91 22.86 0)
+		(unit 1)
+		(body_style 1)
+		(exclude_from_sim no)
+		(in_bom yes)
+		(on_board yes)
+		(in_pos_files yes)
+		(dnp no)
+		(fields_autoplaced yes)
+		(property "Reference" "J103"
+			(at 169.545 15.24 0)
+			(show_name no)
+			(do_not_autoplace no)
+			(effects
+				(font
+					(size 1.27 1.27)
+				)
+			)
+		)
+		(property "Value" "Batt"
+			(at 169.545 17.78 0)
+			(show_name no)
+			(do_not_autoplace no)
+			(effects
+				(font
+					(size 1.27 1.27)
+				)
+			)
+		)
+		(property "Footprint" "Connector_JST:JST_ZH_B4B-ZR_1x04_P1.50mm_Vertical"
+			(at 168.91 22.86 0)
+			(hide yes)
+			(show_name no)
+			(do_not_autoplace no)
+			(effects
+				(font
+					(size 1.27 1.27)
+				)
+			)
+		)
+		(property "Datasheet" ""
+			(at 168.91 22.86 0)
+			(hide yes)
+			(show_name no)
+			(do_not_autoplace no)
+			(effects
+				(font
+					(size 1.27 1.27)
+				)
+			)
+		)
+		(property "Description" "Generic connector, single row, 01x04, script generated"
+			(at 168.91 22.86 0)
+			(hide yes)
+			(show_name no)
+			(do_not_autoplace no)
+			(effects
+				(font
+					(size 1.27 1.27)
+				)
+			)
+		)
+		(pin "4"
+		)
+		(pin "1"
+		)
+		(pin "3"
+		)
+		(pin "2"
+		)
+		(instances
+			(project "sahel_pcb"
+				(path "/e6b0fa3d-63bc-4479-81e5-96b35e896538"
+					(reference "J103")
+					(unit 1)
+				)
+			)
 		)
 	)
@@
 			(effects
 				(font
+					(size 1.27 1.27)
+				)
+				(justify right)
+			)
+		)
+		(pin "Bat_Alert" input
+			(at 91.44 33.02 90)
+			(effects
+				(font
