File: hardware/sahel_pcb_main/sahel_pcb.kicad_pcb (KiCad board)
At the start: 4 copper layers, 90 x 90 mm, 171 parts, among them J101 Conn_02x26_Odd_Even, J102 Conn_02x26_Odd_Even, J301 JTAG_SWD, J302 USB_C_Receptacle_USB2.0_16P, J401 ANT, J501 ANT, SW301 BOOT, SW302 RESET, U201 LMR51430, U202 TPS2116DRL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

Commit message: docs: advance README documentation
Refactor code structure for improved readability and maintainability
Parts:
- added J103: Batt, Connector_JST:JST_ZH_B4B-ZR_1x04_P1.50mm_Vertical, B.Cu at (156.9, 81.0)
- moved D201 0.85 mm to (160.9, 79.6)
- moved R203 0.85 mm to (162.9, 79.6)
Connections:
- net /MCU/I2C1_SCL renamed /_SCL
- net /MCU/I2C1_SDA renamed /_SDA
- U301 pad 1: unconnected-(U301-PE2-Pad1) -> /bat_alert
Routing:
- net /bat_alert: track 0.00 -> 18.8 mm, vias 0 -> 1
- net /_SDA: track 15.3 -> 27.2 mm
- net /_SCL: track 17.1 -> 28.6 mm
- net 3.3V_MAIN: track 58.8 -> 57.9 mm

Commit message: Add support for Sahel STM32H7B0 board and associated drivers
- Created device tree source (DTS) file for Sahel STM32H7B0 board with configurations for GPIO, UART, SPI, I2C, CAN, and various sensors.
- Added YAML configuration for the Sahel STM32H7B0 board, specifying memory and supported features.
- Introduced default configuration file for the board enabling MPU, stack protection, and GPIO.
- Implemented CMake and Kconfig files for BQ76907 battery protection module, including driver source and bindings.
- Added CC1125 radio transceiver module with necessary configurations and driver files.
- Integrated FM24CL64B I2C FRAM module with complete driver implementation and device tree bindings.
- Created example runner script for project execution and setup script for environment preparation.
Parts:
- removed U603: TMP100, Package_TO_SOT_SMD:SOT-23-6
- added U606: RV-8803-C7, Package_SON:MicroCrystal_C7_SON-8_1.5x3.2mm_P0.9mm, F.Cu at (176.8, 76.5)
- U602: value FM24C64C -> FM24CL64B
- U605: value RV-8523-C3 -> TMP112xxDRL; footprint Package_SON:RTC_SMD_MicroCrystal_C3_2.5x3.7mm -> Package_TO_SOT_SMD:SOT-563
- moved U605 10.7 mm to (165.8, 77.4), turned to -90 degrees
- moved C606 7.29 mm to (180.0, 76.4), turned to 0 degrees
- moved R613 4.38 mm to (179.4, 74.2), turned to 90 degrees
- moved C607 2.52 mm to (179.1, 78.3), turned to -90 degrees
- moved R609 1.90 mm to (180.4, 71.4)
- moved R612 0.52 mm to (172.9, 75.8)
- moved C604 0.25 mm to (166.1, 79.6)
Connections:
- U605 pad 1: 3.3V_MAIN -> /_SCL
- U605 pad 2: /MCU/PB5 -> GND
- U605 pad 3: /_SCL -> GND
- U605 pad 4: /_SDA -> GND
- U605 pad 5: /MCU/OSC32_IN -> 3.3V_MAIN
- U605 pad 6: /MCU/PB4 -> /_SDA
Routing:
- net 3.3V_MAIN: track 57.9 -> 48.6 mm
- net /MCU/PB4: track 6.54 -> 13.9 mm, vias 0 -> 2
- net /MCU/OSC32_IN: track 13.2 -> 18.2 mm
- net /_SCL: track 28.6 -> 26.5 mm, vias 0 -> 2
- net /_SDA: track 27.2 -> 26.4 mm
- net /MCU/PB5: vias 0 -> 2

Commit message: chore: bump version to v0.0.2
Parts:
- U401, U501: value CC1125RHBT -> CC1200
Changed lines of the file:
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@@
 			)
 		)
-		(property "Value" "CC1125RHBT"
+		(property "Value" "CC1200"
 			(at 0 3.83 90)
 			(layer "F.Fab")
@@
 			)
 		)
-		(property "Datasheet" "https://www.ti.com/lit/ds/symlink/cc1125.pdf?ts=1775473058389&ref_url=https%253A%252F%252Fwww.google.com%252F"
+		(property "Datasheet" "http://www.ti.com/lit/ds/symlink/cc1200.pdf"
 			(at 0 0 90)
 			(layer "F.Fab")
@@
 			)
 		)
-		(property "SnapEDA_Link" "https://www.snapeda.com/parts/CC1125RHBT/Texas+Instruments/view-part/?ref=snap"
+		(property "SnapEDA_Link" "https://www.snapeda.com/parts/CC1200RHBT/Texas+Instruments/view-part/?ref=snap"
 			(at 0 0 270)
 			(unlocked yes)
@@
 			)
 		)
-		(property "Purchase-URL" "https://www.snapeda.com/api/url_track_click_mouser/?unipart_id=385290&manufacturer=Texas Instruments&part_name=CC1125RHBT&search_term=None"
+		(property "Purchase-URL" "https://www.snapeda.com/api/url_track_click_mouser/?unipart_id=385290&manufacturer=Texas Instruments&part_name=CC1200RHBT&search_term=None"
 			(at 0 0 270)
 			(unlocked yes)
@@
 			)
 		)
-		(property "Check_prices" "https://www.snapeda.com/parts/CC1125RHBT/Texas+Instruments/view-part/?ref=eda"
+		(property "Check_prices" "https://www.snapeda.com/parts/CC1200RHBT/Texas+Instruments/view-part/?ref=eda"
 			(at 0 0 270)
 			(unlocked yes)
@@
 			)
 		)
-		(property "Value" "CC1125RHBT"
+		(property "Value" "CC1200"
 			(at 0 3.83 90)
 			(layer "F.Fab")
@@
 			)
 		)
-		(property "Datasheet" "https://www.ti.com/lit/ds/symlink/cc1125.pdf?ts=1775473058389&ref_url=https%253A%252F%252Fwww.google.com%252F"
+		(property "Datasheet" "http://www.ti.com/lit/ds/symlink/cc1200.pdf"
 			(at 0 0 90)
 			(layer "F.Fab")
@@
 			)
 		)
-		(property "SnapEDA_Link" "https://www.snapeda.com/parts/CC1125RHBT/Texas+Instruments/view-part/?ref=snap"
+		(property "SnapEDA_Link" "https://www.snapeda.com/parts/CC1200RHBT/Texas+Instruments/view-part/?ref=snap"
 			(at 0 0 270)
 			(unlocked yes)
@@
 			)
 		)
-		(property "MP" "CC1125RHBT"
+		(property "MP" "CC1200"
 			(at 0 0 270)
 			(unlocked yes)
@@
 			)
 		)
-		(property "Purchase-URL" "https://www.snapeda.com/api/url_track_click_mouser/?unipart_id=385290&manufacturer=Texas Instruments&part_name=CC1125RHBT&search_term=None"
+		(property "Purchase-URL" "https://www.snapeda.com/api/url_track_click_mouser/?unipart_id=385290&manufacturer=Texas Instruments&part_name=CC1200RHBT&search_term=None"
 			(at 0 0 270)
 			(unlocked yes)
@@
 			)
 		)
-		(property "Check_prices" "https://www.snapeda.com/parts/CC1125RHBT/Texas+Instruments/view-part/?ref=eda"
+		(property "Check_prices" "https://www.snapeda.com/parts/CC1200/Texas+Instruments/view-part/?ref=eda"
 			(at 0 0 270)
 			(unlocked yes)
