File: hardware/sahel_pcb_main/vhf.kicad_sch (KiCad schematic)
At the start: 43 parts, among them J501 ANT, U501 CC1125RHBT, Y501 TG2520SMN-40MHz

Commit message: chore: bump version to v0.0.2
Parts:
- U501: value CC1125RHBT -> CC1200; Check_prices https://www.snapeda.com/parts/CC1125RHBT/Texas+Instruments/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 -> https://www.snapeda.com/parts/CC1200RHBT/Texas+Instruments/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; Purchase-URL https://www.snapeda.com/api/url_track_click_mouser/?unipart_id=385290&manufacturer=Texas Instruments&part_name=CC1125RHBT&search_term=None -> https://www.snapeda.com/api/url_track_click_mouser/?unipart_id=385290&manufacturer=Texas Instruments&part_name=CC1200RHBT&search_term=None; SnapEDA_Link https://www.snapeda.com/parts/CC1125RHBT/Texas+Instruments/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 -> https://www.snapeda.com/parts/CC1200RHBT/Texas+Instruments/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
Changed lines of the file:
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@@
 			)
 		)
-		(property "Value" "CC1125RHBT"
+		(property "Value" "CC1200"
 			(at 120.65 38.1 0)
 			(show_name no)
@@
 			)
 		)
-		(property "Datasheet" "https://www.ti.com/lit/ds/symlink/cc1125.pdf?ts=1775473058389&ref_url=https%253A%252F%252Fwww.google.com%252F"
+		(property "Datasheet" "http://www.ti.com/lit/ds/symlink/cc1200.pdf"
 			(at 120.65 109.22 0)
 			(hide yes)
@@
 			)
 		)
-		(property "SnapEDA_Link" "https://www.snapeda.com/parts/CC1125RHBT/Texas+Instruments/view-part/?ref=snap"
+		(property "SnapEDA_Link" "https://www.snapeda.com/parts/CC1200RHBT/Texas+Instruments/view-part/?ref=snap"
 			(at 120.65 109.22 0)
 			(hide yes)
@@
 			)
 		)
-		(property "Purchase-URL" "https://www.snapeda.com/api/url_track_click_mouser/?unipart_id=385290&manufacturer=Texas Instruments&part_name=CC1125RHBT&search_term=None"
+		(property "Purchase-URL" "https://www.snapeda.com/api/url_track_click_mouser/?unipart_id=385290&manufacturer=Texas Instruments&part_name=CC1200RHBT&search_term=None"
 			(at 120.65 109.22 0)
 			(hide yes)
@@
 			)
 		)
-		(property "Check_prices" "https://www.snapeda.com/parts/CC1125RHBT/Texas+Instruments/view-part/?ref=eda"
+		(property "Check_prices" "https://www.snapeda.com/parts/CC1200RHBT/Texas+Instruments/view-part/?ref=eda"
 			(at 120.65 109.22 0)
 			(hide yes)
